File: pager.kicad_pcb (KiCad board)
At the start: 2 copper layers, 62 x 85 mm, 13 parts, among them J1 Conn_01x18, J2 Conn_01x18, SW1 Up, SW2 Down, SW3 Left, SW4 Right, SW5 Select

Commit message: Add files via upload
Parts:
- moved J2 2.00 mm to (100.0, 102.1)
Changed lines of the file:
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@@
 		(locked yes)
 		(layer "F.Cu")
-		(at 100 104.13 90)
+		(at 100 102.13 90)
 		(descr "Through hole straight socket strip, 1x18, 2.54mm pitch, single row (from Kicad 4.0.7), script generated")
 		(tags "Through hole socket strip THT 1x18 2.54mm single row")
